File: GSLeaf/PCB/GSLeaf.kicad_pcb (KiCad board)
At the start: 2 copper layers, 30 x 103 mm, 119 parts, among them Q1 LED_5050, Q2 IRLML6401, Q3 IRLML6401, Q4 IRLML9303, Q5 2N7002, SW1 SWITCH, SW2 BTN, SW3 BTN, SW4 DIPx6

Commit message: Leaf sent to factory
Parts:
- removed F2, F3, F4, F5, F6, F7: Fuse0R, Resistors:RES_0603_FUSE
- removed SW4: DIPx6, BtnsSwitches:DIP_SMD_1D27X6
- added HOLE1: HOLE_METALLED, PCB:Hole2d4_out4d5mm, F.Cu at (130.6, 61.8)
- added HOLE2: HOLE_METALLED, PCB:Hole2d4_out4d5mm, F.Cu at (130.6, 128.8)
- added HOLE3: HOLE_METALLED, PCB:Hole2d4_out4d5mm, F.Cu at (155.4, 61.8)
- added HOLE4: HOLE_METALLED, PCB:Hole2d4_out4d5mm, F.Cu at (155.4, 128.8)
- moved XL7 21.8 mm to (134.6, 129.5)
- moved R12 8.44 mm to (139.6, 84.6)
- moved SW2 4.70 mm to (132.5, 116.8), turned to 180 degrees
- moved SW3 4.20 mm to (132.5, 123.3)
- moved Logo1 3.81 mm to (139.7, 142.1), turned to 90 degrees
- moved XL5 3.41 mm to (155.7, 68.2)
- moved SW1 3.20 mm to (133.1, 68.0), turned to 180 degrees
- moved C18 0.67 mm to (151.5, 85.0)
- moved XL3 0.60 mm to (156.4, 124.8)
- moved C15 0.58 mm to (150.5, 82.7), turned to 90 degrees
- moved C19 0.50 mm to (141.5, 81.6)
- moved C20 0.50 mm to (143.1, 81.6)
- moved C49 0.41 mm to (132.4, 79.1)
- moved XL2 0.41 mm to (140.1, 63.6)
- moved C52 0.41 mm to (132.4, 77.5)
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Connections:
- DD1 pad 10: /DS1 -> (no net)
- DD1 pad 2: /DS6 -> (no net)
- DD1 pad 3: /DS5 -> (no net)
- DD1 pad 4: /DS4 -> (no net)
- DD1 pad 8: /DS3 -> (no net)
- DD1 pad 9: /DS2 -> (no net)
- Q1 pad 1: GND -> Net-(Q1-Pad1)
- Q1 pad 2: GND -> Net-(Q1-Pad2)
- Q1 pad 3: GND -> Net-(Q1-Pad3)
- Q1 pad 4: Net-(Q1-Pad4) -> GND
- Q1 pad 5: Net-(Q1-Pad5) -> GND
- Q1 pad 6: Net-(Q1-Pad6) -> GND
- R1 pad 1: Net-(Q1-Pad6) -> Net-(Q1-Pad1)
- R2 pad 1: Net-(Q1-Pad5) -> Net-(Q1-Pad2)
- R3 pad 1: Net-(Q1-Pad4) -> Net-(Q1-Pad3)
- XL2 pad H2: Net-(XL2-PadH1) -> (no net)
- XL2 pad H3: Net-(XL2-PadH3) -> (no net)
- XL2 pad H4: Net-(XL2-PadH3) -> Net-(XL2-PadH4)
Routing:
- net GND: track 0.00 -> 648.1 mm, vias 0 -> 116
- net PwrMCU: track 0.00 -> 158.5 mm, vias 0 -> 13
- net /ANT2: track 0.00 -> 142.0 mm
- net VCC: track 0.00 -> 59.9 mm, vias 0 -> 6
- net VAA: track 0.00 -> 58.3 mm, vias 0 -> 5
- net /SDA: track 0.00 -> 51.0 mm, vias 0 -> 4
- net /D-: track 0.00 -> 48.4 mm, vias 0 -> 2
- net /D+: track 0.00 -> 47.4 mm, vias 0 -> 2
- net /SCL: track 0.00 -> 47.2 mm, vias 0 -> 4
- net /ACC_INT1: track 0.00 -> 46.7 mm, vias 0 -> 3
- net /RED_LED: track 0.00 -> 44.7 mm, vias 0 -> 2
- net /GREEN_LED: track 0.00 -> 42.7 mm, vias 0 -> 2
- net +5V: track 0.00 -> 40.4 mm, vias 0 -> 2
- net PwrUnst: track 0.00 -> 38.1 mm, vias 0 -> 1
- net /PWR_CTRLED: track 0.00 -> 32.7 mm, vias 0 -> 2
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- added copper zone on B.Cu, net GND
- added copper zone on F.Cu, net GND
Other:
- outline, holes or cut-outs redrawn
- net class Default: clearance 0.2 -> 0.15; trace_width 0.25 -> 0.15; via_dia 0.8 -> 0.7; via_drill 0.4 -> 0.3
- net class Wide added: clearance 0.15, trace_width 0.5, via_dia 0.7, via_drill 0.3
- rule pad_to_mask_clearance: 0 -> 0.1
- rule trace_clearance: 0.2 -> 0.15
- rule trace_min: 0.2 -> 0.1
- board text added: "+"
- board text added: "-"
- board text added: "Bat measure"
- board text added: "Charger"
- board text added: "GND"
- board text added: "LRCK"
- board text added: "MCLK"
- board text added: "Off On"
- board text added: "Ostranna Quendelasse"
- board text added: "PB13"
- board text added: "PB14"
- board text added: "PB15"
- board text added: "SCLK"
- board text added: "SDIN"
- board text added: "SDOUT"
- board text added: "Speaker"

Commit message: New leaf sch nearly ready
Parts:
- removed ANT1: ANT_PCB_MONO, Radio:ANT_868_SEIDHE
- removed B1: BAT, Installation:EEMB603030
- removed BLN1: BALUN868JOHANSON, Radio:BALUN_JOHANSON868
- removed C1, C11, C20, C3, C36, C48, C49: 10u, Capacitors:CAP_0603
- removed C10, C12, C13, C16, C17, C21, C23, C24, C28, C29, C30, C35, C39, C4, C41, C43, C44, C45, C47, C50, C51, C52, C53: 0.1u, Capacitors:CAP_0603
- removed C14, C22: 22n, Capacitors:CAP_0603
- removed C15, C18, C19, C25, C26, C27, C31, C32, C33, C34, C40, C7: 1u, Capacitors:CAP_0603
- removed C2: 10n, Capacitors:CAP_0603
- removed C37, C38, C5, C6: 18pF, Capacitors:CAP_0603
- removed C42, C46: *, Capacitors:CAP_0402
- removed C8, C9: 150pF, Capacitors:CAP_0603
- removed D1: PMEG2020, Diodes:SOD323
- removed DA1: MCP73832, SOT:SOT23-5
- removed DA2: CS42L52, QFN_DFN:QFN40
- removed DA3: NCP583SQ, SOT:SC82AB
- removed DA4: NCP511SN25, SOT:SOT23-5
- removed DD1: STM32L476Rx, LQFP_TQFP:LQFP64
- removed DD2: CC1101, QFN_DFN:QFN20
- removed DD3: LIS3, LGA:LGA16_3X3_5_3
- removed DD4: MMA8452Q, QFN_DFN:QFN16_5x3
- removed F1: Fuse0R, Resistors:RES_0603_FUSE
- removed HOLE1, HOLE2, HOLE3, HOLE4: HOLE_METALLED, PCB:Hole2d4_out4d5mm
- removed L1: BLM15, Inductors:IND_0402
- removed L2: BLM15AG102SN1, Inductors:IND_0402
- removed L3: *, Inductors:IND_0402
- removed Logo1: Logo, Pictures:Ostranna_12d7_10d1
- removed Q1: LED_5050, LEDs:LED_5050
- removed Q2, Q3: IRLML6401, SOT:SOT23-3
- removed Q4: IRLML9303, SOT:SOT23-3
- removed Q5: 2N7002, SOT:SOT23-3
- removed R1, R2, R3: 100R, Resistors:RES_0603
- removed R10, R11: 51R, Resistors:RES_0603
- removed R12, R4, R9: 10k, Resistors:RES_0603
- removed R13, R14, R17, R18, R19, R5: 100k, Resistors:RES_0603
- removed R15: 20k, Resistors:RES_0603
- removed R16: 56k, Resistors:RES_0603
- removed R6: 1k, Resistors:RES_0603
- removed R7, R8: 4k7, Resistors:RES_0603
- removed SW1: SWITCH, BtnsSwitches:SW_SS-1P2T
- removed SW2, SW3: BTN, BtnsSwitches:BTN_4x4_SMD
- removed TP2, TP3, TP4, TP5, TP6, TP7: TESTPOINT, PCB:TESTPOINT_1MM
- removed XL1: CONN_6, Connectors:PLS-6
- removed XL2: USB_MINI_B, Connectors:USBmicro_MOLEX_WM17142
- removed XL3: CONN_4, Connectors:PLS-4
- removed XL4: AudioJackSimple, Connectors:AUDIO_CKX3_5_30
- removed XL5: CONN_2, Connectors:PLS-2
- removed XL6: CONN_MICROSD, Connectors:MICROSD_CAP_FIX05A
- removed XL7: CONN_1, Connectors:PLS-1Rnd
- removed XTAL1: 12MHz, Quartz:0503x4-4
- removed XTAL2: 27MHz, Quartz:03225C4
Routing:
- net GND: track 648.1 -> 0.00 mm, vias 116 -> 0
- net PwrMCU: track 158.5 -> 0.00 mm, vias 13 -> 0
- net /ANT2: track 142.0 -> 0.00 mm
- net VCC: track 59.9 -> 0.00 mm, vias 6 -> 0
- net VAA: track 58.3 -> 0.00 mm, vias 5 -> 0
- net /SDA: track 51.0 -> 0.00 mm, vias 4 -> 0
- net /D-: track 48.4 -> 0.00 mm, vias 2 -> 0
- net /D+: track 47.4 -> 0.00 mm, vias 2 -> 0
- net /SCL: track 47.2 -> 0.00 mm, vias 4 -> 0
- net /ACC_INT1: track 46.7 -> 0.00 mm, vias 3 -> 0
- net /RED_LED: track 44.7 -> 0.00 mm, vias 2 -> 0
- net /GREEN_LED: track 42.7 -> 0.00 mm, vias 2 -> 0
- net +5V: track 40.4 -> 0.00 mm, vias 2 -> 0
- net PwrUnst: track 38.1 -> 0.00 mm, vias 1 -> 0
- net /PWR_CTRLED: track 32.7 -> 0.00 mm, vias 2 -> 0
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- removed copper zone on B.Cu, net GND
- removed copper zone on F.Cu, net GND
Other:
- board outline removed
- board text removed: "+"
- board text removed: "-"
- board text removed: "Bat measure"
- board text removed: "Charger"
- board text removed: "GND"
- board text removed: "LRCK"
- board text removed: "MCLK"
- board text removed: "Off On"
- board text removed: "Ostranna Quendelasse"
- board text removed: "PB13"
- board text removed: "PB14"
- board text removed: "PB15"
- board text removed: "SCLK"
- board text removed: "SDIN"
- board text removed: "SDOUT"
- board text removed: "Speaker"

Commit message: Layout made by half
Parts:
- added ANT1: ANT_PCB_MONO, Radio:ANT_868_SEIDHE, B.Cu at (135.0, 55.0)
- added B1: BAT, Installation:BATTERY_AAA_X3, F.Cu at (135.0, 81.0)
- added BLN1: BALUN868JOHANSON, Radio:BALUN_JOHANSON868, B.Cu at (142.2, 57.3)
- added C1: 10n, Capacitors:CAP_0603, B.Cu at (175.2, 63.5)
- added C10: 0.1u, Capacitors:CAP_0603, B.Cu at (171.4, 87.8)
- added C11: 0.1u, Capacitors:CAP_0603, B.Cu at (197.8, 116.9)
- added C12: 0.1u, Capacitors:CAP_0603, B.Cu at (179.3, 95.9)
- added C13: 1u, Capacitors:CAP_0603, B.Cu at (180.3, 64.9)
- added C14: 0.1u, Capacitors:CAP_0603, B.Cu at (168.3, 85.7)
- added C15: 22n, Capacitors:CAP_0603, B.Cu at (123.3, 121.1)
- added C16: 1u, Capacitors:CAP_0603, B.Cu at (196.8, 102.3)
- added C17: 0.1u, Capacitors:CAP_0603, B.Cu at (170.0, 64.9)
- added C18: 0.1u, Capacitors:CAP_0603, B.Cu at (197.8, 114.9)
- added C19: 1u, Capacitors:CAP_0603, B.Cu at (178.6, 84.2)
- added C2: 18pF, Capacitors:CAP_0603, B.Cu at (160.5, 116.9)
- added C20: 1u, Capacitors:CAP_0603, B.Cu at (176.3, 61.4)
- added C21: 10u, Capacitors:CAP_0603, B.Cu at (169.6, 79.6)
- added C22: 22n, Capacitors:CAP_0603, B.Cu at (130.0, 120.7)
- added C23: 0.1u, Capacitors:CAP_0603, B.Cu at (171.7, 67.6)
- added C24: 0.1u, Capacitors:CAP_0603, B.Cu at (160.4, 121.0)
- added C25: 0.1u, Capacitors:CAP_0603, B.Cu at (186.3, 102.9)
- added C26: 1u, Capacitors:CAP_0603, B.Cu at (166.7, 74.2)
- added C27: 1u, Capacitors:CAP_0603, B.Cu at (184.3, 69.0)
- added C28: 0.1u, Capacitors:CAP_0603, B.Cu at (164.3, 77.1)
- added C29: 1u, Capacitors:CAP_0603, B.Cu at (166.7, 72.1)
- added C3: 18pF, Capacitors:CAP_0603, B.Cu at (180.7, 101.3)
- added C30: 1u, Capacitors:CAP_0603, B.Cu at (188.0, 94.7)
- added C31: 1u, Capacitors:CAP_0603, B.Cu at (180.3, 67.0)
- added C32: 1u, Capacitors:CAP_0603, B.Cu at (178.6, 86.2)
- added C33: 10u, Capacitors:CAP_0603, B.Cu at (184.7, 73.1)
- added C34: 0.1u, Capacitors:CAP_0603, B.Cu at (168.3, 83.7)
- added C35: 18pF, Capacitors:CAP_0603, B.Cu at (132.2, 64.6)
- added C36: 18pF, Capacitors:CAP_0603, B.Cu at (132.2, 72.4)
- added C37: 18pF, Capacitors:CAP_0603, B.Cu at (135.8, 64.4)
- added C38: 220pF, Capacitors:CAP_0603, B.Cu at (120.7, 59.1)
- added C39: 220pF, Capacitors:CAP_0603, B.Cu at (129.5, 59.1)
- added C4: 0.1u, Capacitors:CAP_0603, B.Cu at (190.3, 107.6)
- added C40: 18pF, Capacitors:CAP_0603, B.Cu at (135.8, 58.7)
- added C41: 0.1u, Capacitors:CAP_0603, B.Cu at (140.8, 67.0)
- added C42: *, Capacitors:CAP_0603, B.Cu at (120.9, 56.5)
- added C43: *, Capacitors:CAP_0603, B.Cu at (129.3, 56.5)
- added C44: 0.1u, Capacitors:CAP_0603, B.Cu at (119.1, 66.6)
- added C45: 10u, Capacitors:CAP_0603, B.Cu at (119.1, 68.2)
- added C46: 0.1u, Capacitors:CAP_0603, B.Cu at (156.3, 103.4)
- added C47: 0.1u, Capacitors:CAP_0603, B.Cu at (127.0, 62.1)
- added C48: *, Capacitors:CAP_0603, B.Cu at (118.6, 55.8)
- added C49: *, Capacitors:CAP_0603, B.Cu at (131.6, 55.8)
- added C5: 1u, Capacitors:CAP_0603, B.Cu at (175.5, 58.8)
- added C50: 1n, Capacitors:CAP_0603, B.Cu at (196.6, 100.2)
- added C51: 0.1u, Capacitors:CAP_0603, B.Cu at (123.0, 62.1)
- added C52: 10u, Capacitors:CAP_0603, B.Cu at (128.6, 62.1)
- added C53: 1n, Capacitors:CAP_0603, B.Cu at (125.0, 62.1)
- added C54: 0.1u, Capacitors:CAP_0603, B.Cu at (126.5, 74.8)
- added C55: 0.1u, Capacitors:CAP_0603, B.Cu at (119.1, 65.0)
- added C56: 1u, Capacitors:CAP_0603, B.Cu at (147.7, 64.4)
- added C57: 10u, Capacitors:CAP_0603, B.Cu at (119.1, 63.4)
- added C58: 0.1u, Capacitors:CAP_0603, B.Cu at (147.7, 59.6)
- added C59: *, Capacitors:CAP_0402, B.Cu at (143.4, 55.6)
- added C6: 150pF, Capacitors:CAP_0603, B.Cu at (179.2, 107.0)
- added C60: 0.1u, Capacitors:CAP_0603, B.Cu at (144.9, 57.6)
- added C61: 0.1u, Capacitors:CAP_0603, B.Cu at (139.5, 57.6)
- added C62: 0.1u, Capacitors:CAP_0603, B.Cu at (138.2, 61.5)
- added C63: *, Capacitors:CAP_0402, B.Cu at (139.0, 55.6)
- added C64: 0.1u, Capacitors:CAP_0603, B.Cu at (142.4, 67.0)
- added C65: 0.1u, Capacitors:CAP_0603, B.Cu at (147.7, 62.8)
- added C66: 10u, Capacitors:CAP_0603, B.Cu at (203.1, 112.8)
- added C67: 10u, Capacitors:CAP_0603, B.Cu at (175.2, 65.5)
- added C68: 0.1u, Capacitors:CAP_0603, B.Cu at (164.3, 79.2)
- added C69: 0.1u, Capacitors:CAP_0603, B.Cu at (184.9, 98.8)
- added C7: 150pF, Capacitors:CAP_0603, B.Cu at (155.0, 118.2)
- added C70: 0.1u, Capacitors:CAP_0603, B.Cu at (197.9, 110.8)
- added C8: 0.1u, Capacitors:CAP_0603, B.Cu at (160.4, 119.0)
- added C9: 10u, Capacitors:CAP_0603, B.Cu at (191.6, 101.5)
- added D1: PMEG2020, Diodes:SOD323, B.Cu at (189.0, 97.9)
- added DA1: CS42L52, QFN_DFN:QFN40, B.Cu at (100.6, 101.0)
- added DA2: NCP583SQ, SOT:SC82AB, B.Cu at (181.8, 89.6)
- added DA3: MCP1700, SOT:SOT23-3, B.Cu at (158.3, 99.6)
- added DA4: NCP511SN25, SOT:SOT23-5, B.Cu at (165.5, 92.0)
- added DD1: STM32L476Rx, LQFP_TQFP:LQFP64, B.Cu at (144.4, 98.7)
- added DD2: PN532, QFN_DFN:QFN40, B.Cu at (125.3, 68.4)
- added DD3: CC1101, QFN_DFN:QFN20, B.Cu at (142.5, 61.7)
- added DD4: LIS3, LGA:LGA16_3X3_5_3, B.Cu at (170.0, 86.1)
- added DD5: MMA8452Q, QFN_DFN:QFN16_5x3, B.Cu at (185.7, 113.3)
- added L1: BLM15, Inductors:IND_0402, B.Cu at (172.8, 76.8)
- added L2: BLM15, Inductors:IND_0402, B.Cu at (173.9, 56.0)
- added L3: 560n, Inductors:IND_0603, B.Cu at (123.4, 58.3)
- added L4: 560n, Inductors:IND_0603, B.Cu at (126.8, 58.3)
- added L5: BLM15AG102SN1, Inductors:IND_0402, B.Cu at (146.8, 66.3)
- added L6: *, Inductors:IND_0402, B.Cu at (141.2, 55.6)
- added Logo1: Logo, Pictures:Ostranna_12d7_10d1, B.Cu at (179.1, 93.2)
- added Q1: LED_5050, LEDs:LED_5050, B.Cu at (135.0, 81.0)
- added Q2: IRLML6401, SOT:SOT23-3, B.Cu at (171.3, 92.1)
- added Q3: IRLML9303, SOT:SOT23-3, B.Cu at (173.1, 71.4)
- added Q4: 2N7002, SOT:SOT23-3, B.Cu at (164.3, 63.2)
- added R1: 100R, Resistors:RES_0603, B.Cu at (171.7, 98.0)
- added R10: 51R, Resistors:RES_0603, B.Cu at (127.7, 121.4)
- added R11: 10k, Resistors:RES_0603, B.Cu at (201.2, 114.9)
- added R12: 100k, Resistors:RES_0603, B.Cu at (164.0, 67.0)
- added R13: 20k, Resistors:RES_0603, B.Cu at (137.8, 65.7)
- added R14: 56k, Resistors:RES_0603, B.Cu at (147.7, 61.2)
- added R15: 100k, Resistors:RES_0603, B.Cu at (175.5, 80.8)
- added R16: 1k, Resistors:RES_0603, B.Cu at (182.9, 71.1)
- added R17: 100k, Resistors:RES_0603, B.Cu at (175.5, 78.7)
- added R18: 100k, Resistors:RES_0603, B.Cu at (172.2, 75.2)
- added R19: 1R, Resistors:RES_0603, B.Cu at (123.2, 55.8)
- added R2: 100R, Resistors:RES_0603, B.Cu at (157.5, 114.9)
- added R20: 1R, Resistors:RES_0603, B.Cu at (127.0, 55.8)
- added R21: 2k7, Resistors:RES_0603, B.Cu at (163.9, 55.2)
- added R3: 100R, Resistors:RES_0603, B.Cu at (163.8, 87.8)
- added R4: 100k, Resistors:RES_0603, B.Cu at (160.7, 91.4)
- added R5: 1k, Resistors:RES_0603, B.Cu at (195.3, 104.3)
- added R6: 10k, Resistors:RES_0603, B.Cu at (182.9, 96.7)
- added R7: 10k, Resistors:RES_0603, B.Cu at (189.9, 103.5)
- added R8: 10k, Resistors:RES_0603, B.Cu at (177.4, 69.0)
- added R9: 51R, Resistors:RES_0603, B.Cu at (123.3, 118.1)
- added SW1: SWITCH, BtnsSwitches:SW_SS-1P2T, F.Cu at (126.4, 113.4)
- added SW2: BTN, BtnsSwitches:BTN_IT1198, F.Cu at (118.3, 109.9)
- added SW3: BTN, BtnsSwitches:BTN_IT1198, F.Cu at (151.6, 109.9)
- added SW4: BTN, BtnsSwitches:BTN_IT1198, F.Cu at (148.2, 119.5)
- added TP1: TESTPOINT, PCB:TESTPOINT_1MM, B.Cu at (168.6, 77.0)
- added TP2: TESTPOINT, PCB:TESTPOINT_1MM, B.Cu at (202.2, 110.3)
- added XL1: CONN_6, Connectors:PLS-6, B.Cu at (155.0, 81.8)
- added XL2: USB_MINI_B, Connectors:USBmicro_MOLEX_1050170001, F.Cu at (139.0, 127.0)
- added XL3: AudioJackSimple, Connectors:AUDIO_CKX3_5_30, F.Cu at (127.6, 127.0)
- added XL4: CONN_MICROSD, Installation:MICROSD_CAP_FIX05A, F.Cu at (138.2, 114.4)
- added XL5: CONN_1, Connectors:PLS-1Rnd, F.Cu at (149.6, 114.5)
- added XTAL1: 12MHz, Quartz:0503x4-4, B.Cu at (144.2, 87.6)
- added XTAL2: 27.12MHz, Quartz:0503x4-4, B.Cu at (132.2, 68.5)
- added XTAL3: 27MHz, Quartz:03225C4, B.Cu at (135.8, 61.5)
Other:
- board outline added: 46 x 103 mm

Commit message: Layout done
Parts:
- Logo1: moved to F.Cu
- moved C18 81.0 mm to (118.6, 98.0), turned to 180 degrees
- moved C16 77.5 mm to (119.3, 101.9), turned to 90 degrees
- moved TP2 76.4 mm to (137.9, 68.9)
- moved C50 76.0 mm to (132.3, 59.7), turned to 90 degrees
- moved C31 72.1 mm to (123.7, 111.7), turned to 180 degrees
- moved C27 71.2 mm to (118.6, 96.4), turned to 180 degrees
- moved C70 70.0 mm to (137.7, 75.0), turned to 180 degrees
- moved C33 68.3 mm to (125.5, 107.2), turned to 90 degrees
- moved Logo1 68.3 mm to (135.1, 41.0)
- moved C1 67.2 mm to (136.6, 118.5)
- moved C66 66.9 mm to (151.8, 69.9), turned to 90 degrees
- moved L2 66.3 mm to (128.5, 104.3), turned to 90 degrees
- moved C20 65.8 mm to (118.6, 93.2)
- moved R11 64.6 mm to (136.6, 116.9)
- moved R8 62.1 mm to (142.8, 120.6)
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
Commit message: Tracing in progress
Other:
- net class Ant added: clearance 0.2, trace_width 0.3, via_dia 0.7, via_drill 0.3
Changed lines of the file:
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@@
     (links 394)
     (no_connects 393)
-    (area 111.961059 23.949999 158.032843 130.024011)
+    (area 111.961059 23.949999 158.032843 130.074011)
     (thickness 1.6)
     (drawings 55)
@@
     (uvia_dia 0.3)
     (uvia_drill 0.1)
-    (add_net +3.3V)
-    (add_net +5V)
-    (add_net +BATT)
     (add_net /ACC_INT1)
     (add_net /ACC_PWR)
@@
     (add_net /AU_SDIN)
     (add_net /AU_SDOUT)
-    (add_net /Antenna)
     (add_net /BAT_MEAS)
     (add_net /BLUE_LED)
@@
     (add_net /PN_RESET)
     (add_net /PN_SCK)
-    (add_net /PN_VDD)
-    (add_net /PWR_UNST_ALWAYS)
     (add_net /RED_LED)
     (add_net /RF1)
@@
     (add_net /SD_DAT2)
     (add_net /SD_DAT3)
-    (add_net /SD_PWR)
     (add_net /SD_PWR_EN)
     (add_net /SWCLK)
@@
     (add_net /UART_RX)
     (add_net /UART_TX)
-    (add_net GND)
     (add_net "Net-(C15-Pad1)")
     (add_net "Net-(C16-Pad1)")
@@
     (add_net "Net-(XL2-PadH3)")
     (add_net "Net-(XL2-PadH4)")
-    (add_net PwrMCU)
-    (add_net PwrUnst)
-    (add_net VAA)
-    (add_net VCC)
+  )
+  (net_class Ant ""
+    (clearance 0.2)
+    (trace_width 0.3)
+    (via_dia 0.7)
+    (via_drill 0.3)
+    (uvia_dia 0.3)
+    (uvia_drill 0.1)
+    (add_net /Antenna)
   )
   (net_class Wide ""
@@
     (uvia_dia 0.3)
     (uvia_drill 0.1)
+    (add_net +3.3V)
+    (add_net +5V)
+    (add_net +BATT)
+    (add_net /PN_VDD)
+    (add_net /PWR_UNST_ALWAYS)
+    (add_net /SD_PWR)
+    (add_net GND)
+    (add_net PwrMCU)
+    (add_net PwrUnst)
+    (add_net VAA)
+    (add_net VCC)
   )
   (module Installation:BATTERY_AAA_X3 (layer F.Cu)

Commit message: Sent to factory
Parts:
- moved TP1 4.47 mm to (134.2, 98.1)
- moved C1 1.30 mm to (136.7, 119.8)
- moved R11 1.30 mm to (136.7, 118.2)
- moved C54 1.20 mm to (127.3, 73.9), turned to 0 degrees
- moved C16 0.60 mm to (119.3, 102.5)
- moved L2 0.30 mm to (128.5, 104.6)
- moved R13 0.28 mm to (138.1, 65.7)
Routing:
- net GND: track 0.00 -> 758.8 mm, vias 0 -> 138
- net /Antenna: track 0.00 -> 393.1 mm, vias 0 -> 8
- net /ANT2: track 0.00 -> 141.3 mm
- net PwrMCU: track 0.00 -> 89.5 mm, vias 0 -> 6
- net PwrUnst: track 0.00 -> 80.2 mm, vias 0 -> 1
- net +3.3V: track 0.00 -> 73.1 mm, vias 0 -> 2
- net /SDA: track 0.00 -> 64.3 mm, vias 0 -> 3
- net /SCL: track 0.00 -> 63.3 mm, vias 0 -> 3
- net VCC: track 0.00 -> 61.2 mm, vias 0 -> 6
- net /AU_RST: track 0.00 -> 49.3 mm, vias 0 -> 2
- net VAA: track 0.00 -> 48.2 mm, vias 0 -> 4
- net /PN_SCK: track 0.00 -> 41.3 mm, vias 0 -> 2
- net /PN_MISO: track 0.00 -> 40.5 mm, vias 0 -> 2
- net /CC_CS: track 0.00 -> 40.5 mm, vias 0 -> 2
- net /PN_NSS: track 0.00 -> 40.1 mm, vias 0 -> 2
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- added copper zone on B.Cu, net GND
- added copper zone on F.Cu, net GND
Other:
- board text added: "Audio"
- board text added: "GND"
- board text added: "NFC"
- board text added: "Ostranna"
- board text added: "Quendelasse v2"
- board text added: "Radio"
