File: GSLeaf/PCB/GSLeaf.sch (KiCad schematic (older format))
At the start: 119 parts, among them Q1 LED_5050, Q2 IRLML6401, Q3 IRLML6401, Q4 IRLML9303, Q5 2N7002, SW1 SWITCH, SW2 BTN, SW3 BTN, SW4 DIPx6

Commit message: Leaf sent to factory
Parts:
- removed F2, F3, F4, F5, F6, F7: Fuse0R, Resistors:RES_0603_FUSE, symbol Fuse0R
- removed SW4: DIPx6, BtnsSwitches:DIP_SMD_1D27X6, symbol DIPx6
- added HOLE1, HOLE2, HOLE3, HOLE4: HOLE_METALLED, PCB:Hole2d4_out4d5mm, symbol HOLE_METALLED
Connections:
- net labels removed: DS1, DS2, DS3, DS4, DS5, DS6
- wire segments 404 -> 371
- no-connect marks 21 -> 31

Commit message: + Antenna matched
Parts:
- C42: value * -> DoNotMount
- C46: value * -> 3pF
- L3: value * -> 12nH
Changed lines of the file:
@@
 P 19550 2650
 F 0 "L3" V 19450 2510 40  0000 C CNN
-F 1 "*" V 19450 2650 40  0000 C CNN
+F 1 "12nH" V 19450 2650 40  0000 C CNN
 F 2 "Inductors:IND_0402" V 19610 2660 40  0001 C CNN
 F 3 "" V 19450 2510 60  0001 C CNN
@@
 P 19200 3150
 F 0 "C42" H 19100 3050 50  0000 L CNN
-F 1 "*" H 19100 3250 50  0000 L CNN
+F 1 "DoNotMount" H 19100 3250 50  0000 L CNN
 F 2 "Capacitors:CAP_0402" V 19300 3000 28  0001 C BNN
 F 3 "" H 19100 3050 60  0001 C CNN
@@
 P 19900 3150
 F 0 "C46" H 19800 3050 50  0000 L CNN
-F 1 "*" H 19800 3250 50  0000 L CNN
+F 1 "3pF" H 19800 3250 50  0000 L CNN
 F 2 "Capacitors:CAP_0402" V 20000 3000 28  0001 C BNN
 F 3 "" H 19800 3050 60  0001 C CNN

Commit message: New leaf sch nearly ready
Parts:
- removed C1, C3: 10u, Capacitors:CAP_0603, symbol C
- removed DA1: MCP73832, SOT:SOT23-5, symbol MCP73832
- removed F1: Fuse0R, Resistors:RES_0603_FUSE, symbol Fuse0R
- removed Q3: IRLML6401, SOT:SOT23-3, symbol P_3PIN
- removed R13: 100k, Resistors:RES_0603, symbol R
- removed R4: 10k, Resistors:RES_0603, symbol R
- removed TP2, TP3, TP4, TP6: TESTPOINT, PCB:TESTPOINT_1MM, symbol TESTPOINT
- removed XL3: CONN_4, Connectors:PLS-4, symbol CONN_4
- removed XL5: CONN_2, Connectors:PLS-2, symbol CONN_2
- added C35, C36: 18pF, Capacitors:CAP_0603, symbol C
- added C38, C39: 220pF, Capacitors:CAP_0603, symbol C
- added C42, C43, C48, C49: *, Capacitors:CAP_0603, symbol C
- added C44, C46, C47, C51, C54, C55: 0.1u, Capacitors:CAP_0603, symbol C
- added C45, C52, C57: 10u, Capacitors:CAP_0603, symbol C
- added C50, C53: 1n, Capacitors:CAP_0603, symbol C
- added DA3: MCP1700, SOT:SOT23-3, symbol MCP1700
- added DD2: PN532, symbol PN532
- added L2, L3: 560n, Inductors:IND_0603, symbol L
- added R16: 1k, Resistors:RES_0603, symbol R
- added R19, R20: 1R, Resistors:RES_0603, symbol R
- added R21: 2k7, Resistors:RES_0603, symbol R
- added XTAL2: 27.12MHz, Quartz:0503x4-4, symbol CRYSTAL_H
- R6: renamed from R7; value 4k7 -> 10k
- R7: renamed from R8; value 4k7 -> 10k
- renumbered C2 to C1, C12 to C10, C13 to C11, C21 to C12, C25 to C13, C28 to C14, C14 to C15, C15 to C16, C16 to C17, C17 to C18, C18 to C19, C5 to C2, C19 to C20, C20 to C21, C29 to C25, C30 to C28, C31 to C29, C6 to C3, C32 to C30, C34 to C31, C33 to C32, C36 to C33, C35 to C34, C38 to C40, C39 to C41, C7 to C5, C40 to C56, C41 to C58, C42 to C59, C8 to C6, C43 to C60, C44 to C61, C45 to C62, C46 to C63, C47 to C64, C50 to C65, C48 to C66, C49 to C67, C51 to C68, C52 to C69, C9 to C7, C53 to C70, C10 to C8, C11 to C9, DA2 to DA1, DA3 to DA2, DD2 to DD3, DD3 to DD4, DD4 to DD5, L2 to L4, L3 to L5, Q4 to Q3, Q5 to Q4, R11 to R10, R12 to R11, R14 to R12, R15 to R13, R16 to R14, R17 to R15, R18 to R17, R19 to R18, R5 to R4, R6 to R5, R9 to R8, R10 to R9, TP5 to TP1, TP7 to TP2, XL4 to XL3, XL6 to XL4, XL7 to XL5, XTAL2 to XTAL3
Connections:
- net labels added: ANT01, ANT02, Antenna, PN_IRQ, PN_MISO, PN_MOSI, PN_NSS, PN_RESET, PN_SCK, PN_VDD, RX_NET
- net labels removed: Charge, PWR_CTRLED, PWR_EN, SPK_M, SPK_P
- wire segments 371 -> 432
- no-connect marks 31 -> 46
Other:
- note added: "Antenna"
- note added: "Damping Resistors"
- note added: "EMC Filter"
- note added: "Matching Circuit"
- note added: "One or another"
- note added: "PN"
- note added: "SPI Mode"
- note removed: "Just\npins"
- note removed: "Li-Ion charger\n10k => 120mA"
- note removed: "Maybe transistor is not needed"

Commit message: Layout made by half
Parts:
- removed HOLE1, HOLE2, HOLE3, HOLE4: HOLE_METALLED, PCB:Hole2d4_out4d5mm, symbol HOLE_METALLED
- added L2: BLM15, Inductors:IND_0402, symbol L
- added SW4: BTN, BtnsSwitches:BTN_IT1198, symbol BUTTON
- B1: footprint Installation:EEMB603030 -> Installation:BATTERY_AAA_X3
- C59: value DoNotMount -> *
- C63: value 3pF -> *
- DD2: footprint (none) -> QFN_DFN:QFN40
- L6: renamed from L5; value 12nH -> *
- SW2, SW3: footprint BtnsSwitches:BTN_4x4_SMD -> BtnsSwitches:BTN_IT1198
- XL2: footprint Connectors:USBmicro_MOLEX_WM17142 -> Connectors:USBmicro_MOLEX_1050170001
- XL4: footprint Connectors:MICROSD_CAP_FIX05A -> Installation:MICROSD_CAP_FIX05A
- renumbered L2 to L3, L3 to L4, L4 to L5
Connections:
- net labels added: ACC_PWR, BTN_COM
- wire segments 432 -> 431
- no-connect marks 46 -> 48

Commit message: Tracing in progress
Changed lines of the file:
@@
 Text Label 19750 9750 0    60   ~ 0
 SDA
-$Comp
-L PwrMCU #PWR0107
-U 1 1 593BAE6E
-P 19900 9850
-F 0 "#PWR0107" H 19900 9900 30  0001 C CNN
-F 1 "PwrMCU" H 19970 9880 30  0000 C CNN
-F 2 "" H 19900 9850 60  0000 C CNN
-F 3 "" H 19900 9850 60  0000 C CNN
-	1    19900 9850
-	-1   0    0    -1
-$EndComp
-Wire Wire Line
-	19900 9850 20200 9850
+Wire Wire Line
+	19650 9850 20200 9850
 $Comp
 L PwrMCU #PWR0108
@@
 Text Label 22400 7450 0    60   ~ 0
 ACC_PWR
+Text Label 19650 9850 0    60   ~ 0
+ACC_PWR
 $EndSCHEMATC

Commit message: * First commit of new system (17.6.0) on new board. Uart works.
Parts:
- C42: value * -> 30pF
- C48: value * -> 220+47+20pF
Changed lines of the file:
@@
 P 16100 10950
 F 0 "C42" V 16050 10800 50  0000 C CNN
-F 1 "*" V 16050 11050 50  0000 C CNN
+F 1 "30pF" V 16050 11050 50  0000 C CNN
 F 2 "Capacitors:CAP_0603" V 16200 10800 28  0001 C BNN
 F 3 "" H 16000 10850 60  0001 C CNN
@@
 P 16850 11250
 F 0 "C48" H 16800 11100 50  0000 C CNN
-F 1 "*" H 16800 11350 50  0000 C CNN
+F 1 "220+47+20pF" H 16800 11350 50  0000 C CNN
 F 2 "Capacitors:CAP_0603" V 16950 11100 28  0001 C BNN
 F 3 "" H 16750 11150 60  0001 C CNN
