File: GSLeaf/PCB/GSLeaf.sch (KiCad schematic (older format))
At the start: 116 parts, among them Q1 LED_5050, Q2 IRLML6401, Q3 IRLML6401, Q4 IRLML9303, Q5 2N7002, SW1 SWITCH, SW2 BTN, SW3 BTN

Commit message: Switching to allnew
Parts:
- ANT1: symbol ANT_PCB_MONO -> Antennas_kl:ANT_PCB_MONO
- B1: symbol BAT -> Power_kl:BAT
- BLN1: symbol BALUN868JOHANSON -> RF_ICs:BALUN868JOHANSON
- C1, C10, C11, C12, C13, C14, C15, C16, C17, C18, C19, C2, C20, C21, C22, C23, C24, C25, C26, C27, C28, C29, C3, C30, C31, C32, C33, C34, C35, C36, C37, C38, C39, C4, C40, C41, C42, C43, C44, C45, C46, C47, C48, C49, C5, C50, C51, C52, C53, C6, C7, C8, C9: symbol C -> Tittar_kl:C
- D1: symbol D_Shottky -> Tittar_kl:D_Shottky
- DA1: symbol MCP73832 -> Power_kl:MCP73832
- DA2: symbol CS42L52 -> Audio_kl:CS42L52
- DA3: symbol NCP583SQ -> Power_kl:NCP583SQ
- DA4: symbol TPS763xx -> Power_kl:TPS763xx
- DD1: symbol STM32L476Rx -> st_kl:STM32L476Rx
- DD2: symbol CC1101 -> RF_ICs:CC1101
- DD3: symbol LIS3 -> Sensors:LIS3
- DD4: symbol MMA8452Q -> Sensors:MMA8452Q
- F1: symbol Fuse0R -> Tittar_kl:Fuse0R
- HOLE1, HOLE2, HOLE3, HOLE4: symbol HOLE_METALLED -> pcb_details:HOLE_METALLED
- L1, L2, L3: symbol L -> Tittar_kl:L
- Logo1: symbol Logo -> pcb_details:Logo
- Q1: symbol LED_5050 -> Tittar_kl:LED_5050
- Q2, Q3, Q4: symbol P_3PIN -> Transistors_kl:P_3PIN
- Q5: symbol N_3PIN -> Transistors_kl:N_3PIN
- R1, R10, R11, R12, R13, R14, R15, R16, R17, R18, R19, R2, R3, R4, R5, R6, R7, R8, R9: symbol R -> Tittar_kl:R
- SW1: symbol SWITCH -> Switches:SWITCH_1P2T
- SW2, SW3: symbol BUTTON -> Switches:BUTTON
- TP2, TP3, TP4, TP5, TP6, TP7: symbol TESTPOINT -> pcb_details:TESTPOINT
- XL1: symbol CONN_6 -> Connectors_kl:CONN_6
- XL2: symbol USB_MINI_B -> Connectors_kl:USB_MINI_B
- XL3: symbol CONN_4 -> Connectors_kl:CONN_4
- XL4: symbol AudioJackSimple -> Connectors_kl:AudioJackSimple
- XL5: symbol CONN_2 -> Connectors_kl:CONN_2
- XL6: symbol CONN_MICROSD -> Connectors_kl:CONN_MICROSD
- XL7: symbol CONN_1 -> Connectors_kl:CONN_1
- XTAL1, XTAL2: symbol CRYSTAL_H -> Tittar_kl:CRYSTAL_H
Connections:
- net labels added: +3v3
- net labels removed: +3.3V
- wire segments 371 -> 471
